File: controller-ha-v1.brd (EAGLE design)
At the start: 188 x 169.5 mm, 138 parts, among them U1 DS1307, U2 ARDUINO-MEGAPRO-5V, U3 ARDUINO-MEGAFULL

Commit message: Submit all new design
Adding version 3-4 for driver & controller; Adding version 1-2 IO Module
Parts:
- removed C9-100N1, C9-100N10, C9-100N11, C9-100N12, C9-100N13, C9-100N14, C9-100N15, C9-100N16, C9-100N17, C9-100N18, C9-100N19, C9-100N2, C9-100N20, C9-100N21, C9-100N22, C9-100N23, C9-100N24, C9-100N25, C9-100N26, C9-100N3, C9-100N4, C9-100N5, C9-100N6, C9-100N7, C9-100N8, C9-100N9: (no value), rcl:C0603
- removed CN1: (no value), adafruit:DCJACK_2MM_PTH
- removed U$1: DCDCMODULE, bontor:DCDCMODULE
- removed U2: ARDUINO-MEGAPRO-5V, SparkFun-Boards:ARDUINO_MEGA-PRO-5V
- moved C11-22P 16.2 mm to (40.9, 23.8)
- moved R1-1K 16.2 mm to (36.1, 39.4)
- moved R30 16.2 mm to (30.4, 24.5)
- moved R9-22 16.2 mm to (38.1, 17.9)
- moved U$5 16.2 mm to (30.8, 10.4)
- moved BAT1 16.2 mm to (96.8, 31.5)
- moved C10-4U7 16.2 mm to (49.9, 26.4)
- moved C7-100U 16.2 mm to (64.7, 44.8)
- moved C8-100U 16.2 mm to (64.5, 52.3)
- moved CSIM_100N 16.2 mm to (43.9, 14.9)
- moved CSIM_22P 16.2 mm to (38.1, 14.8)
- moved D15 16.2 mm to (44.4, 19.1)
- moved JP1 16.2 mm to (33.9, 9.12)
- moved LED1 16.2 mm to (67.4, 10.5)
- moved LED2 16.2 mm to (61.6, 10.5)
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Connections:
- net +3V3: no longer U$1.VOUT
- net GND: no longer C9-100N1.1, C9-100N10.1, C9-100N11.1, C9-100N12.1, C9-100N13.1, C9-100N14.1, C9-100N15.1, C9-100N16.1, C9-100N17.1, C9-100N18.1, C9-100N19.1, C9-100N2.1, C9-100N20.1, C9-100N21.1, C9-100N22.1, C9-100N23.1, C9-100N24.1, C9-100N25.1, C9-100N26.1, C9-100N3.1, C9-100N4.1, C9-100N5.1, C9-100N6.1, C9-100N7.1, C9-100N8.1, C9-100N9.1, CN1.GND, CN1.GNDBREAK, U$1.GND#0, U$1.GND#1
- net N$17: now also AC_IN.3; no longer AC_IN.1
- net N$7: now also AC_IN.1; no longer AC_IN.3
- net VCC: no longer C9-100N1.2, C9-100N10.2, C9-100N11.2, C9-100N12.2, C9-100N13.2, C9-100N14.2, C9-100N15.2, C9-100N16.2, C9-100N17.2, C9-100N18.2, C9-100N19.2, C9-100N2.2, C9-100N20.2, C9-100N21.2, C9-100N22.2, C9-100N23.2, C9-100N24.2, C9-100N25.2, C9-100N26.2, C9-100N3.2, C9-100N4.2, C9-100N5.2, C9-100N6.2, C9-100N7.2, C9-100N8.2, C9-100N9.2, CN1.PWR, U$1.VIN
Routing:
- net VCC: track 1689.2 -> 1329.4 mm, vias 29 -> 14
- net SR_DS: track 302.3 -> 0.00 mm, vias 2 -> 0
- net SHCP: track 350.0 -> 186.0 mm
- net SR_RST: track 331.8 -> 168.7 mm, vias 14 -> 13
- net STCP: track 364.0 -> 201.6 mm
- net DS_OE: track 367.1 -> 210.5 mm
- net GND: track 1236.8 -> 1097.1 mm, vias 73 -> 50
- net N$55: track 89.0 -> 0.00 mm
- net N$43: track 89.0 -> 0.00 mm
- net SCL: track 87.2 -> 20.4 mm
- net SDA: track 90.2 -> 26.2 mm, vias 1 -> 0
- net Q7: track 91.0 -> 106.0 mm
- net CLK: track 256.9 -> 271.9 mm
- net CE: track 208.9 -> 196.6 mm
- net N$7: track 25.7 -> 33.0 mm
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- removed copper zone on layer 1, net GND
- removed copper zone on layer 16, net GND
- removed copper zone on layer 1, net VCC
Other:
- board size 188 x 169.5 mm -> 181.2 x 176.6 mm
