File: IO_board-ha-v2.brd (EAGLE design)
At the start: 99 x 102 mm, 45 parts, among them J1 4-PIN-CON-1759017, J2 4-PIN-CON-1759017

Commit message: change in controller design
Change component position & adding hole to controller design
Parts:
- R1, R2, R3, R4, R5, R6, R7, R8, RN1, RN2, RN4, RN5: value (none) -> 10K
Changed lines of the file:
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@@
 <layer number="25" name="tNames" color="7" fill="1" visible="yes" active="yes"/>
 <layer number="26" name="bNames" color="7" fill="1" visible="yes" active="yes"/>
-<layer number="27" name="tValues" color="7" fill="1" visible="yes" active="yes"/>
-<layer number="28" name="bValues" color="7" fill="1" visible="yes" active="yes"/>
+<layer number="27" name="tValues" color="7" fill="1" visible="no" active="yes"/>
+<layer number="28" name="bValues" color="7" fill="1" visible="no" active="yes"/>
 <layer number="29" name="tStop" color="7" fill="3" visible="no" active="yes"/>
 <layer number="30" name="bStop" color="7" fill="6" visible="no" active="yes"/>
@@
 <element name="SHIFT1" library="74xx-eu" package="SO16" value="74HC165D" x="24.16" y="19.06" rot="R180"/>
 <element name="SHIFT2" library="74xx-eu" package="SO16" value="74HC165D" x="24.21" y="56.53" rot="R180"/>
-<element name="RN1" library="resistor-net" package="RN-9" value="" x="11.75" y="19.77" rot="R90">
+<element name="RN1" library="resistor-net" package="RN-9" value="10K" x="11.75" y="19.77" rot="R90">
 <attribute name="OC_NEWARK" value="unknown" x="11.75" y="19.77" size="1.778" layer="27" rot="R90" display="off"/>
 <attribute name="MPN" value="" x="11.75" y="19.77" size="1.778" layer="27" rot="R90" display="off"/>
@@
 <element name="SHIFT4" library="74xx-eu" package="SO16" value="74HC165D" x="72" y="57.08"/>
 <element name="SHIFT5" library="74xx-eu" package="SO16" value="74HC165D" x="71.72" y="16.41"/>
-<element name="RN2" library="resistor-net" package="RN-9" value="" x="11.66" y="63.77" rot="R90">
+<element name="RN2" library="resistor-net" package="RN-9" value="10K" x="11.66" y="63.77" rot="R90">
 <attribute name="OC_NEWARK" value="unknown" x="11.66" y="63.77" size="1.6764" layer="27" rot="R90" display="off"/>
 <attribute name="MPN" value="" x="11.66" y="63.77" size="1.6764" layer="27" rot="R90" display="off"/>
@@
 <attribute name="OC_FARNELL" value="unknown" x="11.66" y="63.77" size="1.6764" layer="27" rot="R90" display="off"/>
 </element>
-<element name="RN4" library="resistor-net" package="RN-9" value="" x="87.42" y="72.39" rot="R90">
+<element name="RN4" library="resistor-net" package="RN-9" value="10K" x="87.42" y="72.39" rot="R90">
 <attribute name="OC_NEWARK" value="unknown" x="87.42" y="72.39" size="1.6764" layer="27" rot="R90" display="off"/>
 <attribute name="MPN" value="" x="87.42" y="72.39" size="1.6764" layer="27" rot="R90" display="off"/>
@@
 <attribute name="OC_FARNELL" value="unknown" x="87.42" y="72.39" size="1.6764" layer="27" rot="R90" display="off"/>
 </element>
-<element name="RN5" library="resistor-net" package="RN-9" value="" x="87.57" y="28.39" rot="R90">
+<element name="RN5" library="resistor-net" package="RN-9" value="10K" x="87.57" y="28.39" rot="R90">
 <attribute name="OC_NEWARK" value="unknown" x="87.57" y="28.39" size="1.6764" layer="27" rot="R90" display="off"/>
 <attribute name="MPN" value="" x="87.57" y="28.39" size="1.6764" layer="27" rot="R90" display="off"/>
@@
 <element name="C2" library="resistor" package="C0805" value="100nF" x="11.6" y="50.3" rot="R270"/>
 <element name="C3" library="resistor" package="C0805" value="100nF" x="46.4" y="48.7"/>
-<element name="C4" library="resistor" package="C0805" value="100nF" x="87.5" y="58.4" rot="R270"/>
+<element name="C4" library="resistor" package="C0805" value="100nF" x="87.5" y="58.4" smashed="yes" rot="R270">
+<attribute name="NAME" x="88.516" y="59.289" size="1.27" layer="25" rot="R270"/>
+<attribute name="VALUE" x="85.214" y="59.289" size="1.27" layer="27" rot="R270"/>
+</element>
 <element name="C5" library="resistor" package="C0805" value="100nF" x="87.5" y="14.9" rot="MR270"/>
-<element name="C6" library="resistor" package="C0805" value="100nF" x="83.2" y="58.6" rot="R90"/>
+<element name="C6" library="resistor" package="C0805" value="100nF" x="83.2" y="58.6" smashed="yes" rot="R90">
+<attribute name="NAME" x="82.184" y="57.711" size="1.27" layer="25" rot="R90"/>
+<attribute name="VALUE" x="85.486" y="57.711" size="1.27" layer="27" rot="R90"/>
+</element>
 <element name="C7" library="resistor" package="C0805" value="100nF" x="26" y="43" rot="MR0"/>
 <element name="C8" library="resistor" package="C0805" value="100nF" x="48.4" y="58.9"/>
 <element name="C9" library="resistor" package="C0805" value="100nF" x="20.4" y="73.9" rot="MR180"/>
 <element name="C10" library="resistor" package="C0805" value="100nF" x="81.2" y="22.6" rot="R90"/>
-<element name="R1" library="resistor" package="R0603" value="" x="85.1" y="87.7" rot="R180"/>
-<element name="R2" library="resistor" package="R0603" value="" x="84.4" y="85.1" rot="R180"/>
-<element name="R3" library="resistor" package="R0603" value="" x="86.64" y="43.6" rot="R180"/>
-<element name="R4" library="resistor" package="R0603" value="" x="85.9" y="41" rot="R180"/>
-<element name="R5" library="resistor" package="R0603" value="" x="22.3" y="48.8" rot="R270"/>
-<element name="R6" library="resistor" package="R0603" value="" x="24" y="48.8" rot="R270"/>
-<element name="R7" library="resistor" package="R0603" value="" x="12" y="76.5"/>
-<element name="R8" library="resistor" package="R0603" value="" x="12.8" y="81.1"/>
+<element name="R1" library="resistor" package="R0603" value="10K" x="85.1" y="87.7" rot="R180"/>
+<element name="R2" library="resistor" package="R0603" value="10K" x="84.4" y="85.1" rot="R180"/>
+<element name="R3" library="resistor" package="R0603" value="10K" x="86.64" y="43.6" rot="R180"/>
+<element name="R4" library="resistor" package="R0603" value="10K" x="85.9" y="41" rot="R180"/>
+<element name="R5" library="resistor" package="R0603" value="10K" x="22.3" y="48.8" rot="R270"/>
+<element name="R6" library="resistor" package="R0603" value="10K" x="24" y="48.8" rot="R270"/>
+<element name="R7" library="resistor" package="R0603" value="10K" x="12" y="76.5"/>
+<element name="R8" library="resistor" package="R0603" value="10K" x="12.8" y="81.1"/>
 <element name="JP1" library="SparkFun-Connectors" package="2X5-SHROUDED" value="" x="46.9" y="14.8" rot="R270"/>
 <element name="JP2" library="SparkFun-Connectors" package="2X5-SHROUDED" value="" x="48.2" y="86.7" rot="R270"/>
