File: IO_board-ha-v2.sch (EAGLE design)
At the start: 45 parts, among them J1 4-PIN-CON-1759017, J2 4-PIN-CON-1759017

Commit message: change in controller design
Change component position & adding hole to controller design
Parts:
- R1, R2, R3, R4, R5, R6, R7, R8, RN1, RN2, RN4, RN5: value (none) -> 10K
Changed lines of the file:
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@@
 <part name="GND29" library="supply1" deviceset="GND" device=""/>
 <part name="P+13" library="SparkFun" deviceset="VCC" device=""/>
-<part name="RN1" library="resistor-net" deviceset="RN08" device=""/>
+<part name="RN1" library="resistor-net" deviceset="RN08" device="" value="10K"/>
 <part name="P+8" library="SparkFun" deviceset="VCC" device=""/>
 <part name="SHIFT3" library="74xx-eu" deviceset="74*165" device="D" technology="HC" value="74HC165D"/>
@@
 <part name="GND26" library="supply1" deviceset="GND" device=""/>
 <part name="P+15" library="SparkFun" deviceset="VCC" device=""/>
-<part name="RN2" library="resistor-net" deviceset="RN08" device=""/>
+<part name="RN2" library="resistor-net" deviceset="RN08" device="" value="10K"/>
 <part name="P+34" library="SparkFun" deviceset="VCC" device=""/>
-<part name="RN4" library="resistor-net" deviceset="RN08" device=""/>
+<part name="RN4" library="resistor-net" deviceset="RN08" device="" value="10K"/>
 <part name="P+36" library="SparkFun" deviceset="VCC" device=""/>
-<part name="RN5" library="resistor-net" deviceset="RN08" device=""/>
+<part name="RN5" library="resistor-net" deviceset="RN08" device="" value="10K"/>
 <part name="P+37" library="SparkFun" deviceset="VCC" device=""/>
 <part name="SHIFTOUTA" library="74xx-eu" deviceset="74*595" device="D" technology="HC"/>
@@
 <part name="P+26" library="supply1" deviceset="+12V" device=""/>
 <part name="GND8" library="supply1" deviceset="GND" device=""/>
-<part name="R1" library="resistor" deviceset="R-EU_" device="R0603"/>
-<part name="R2" library="resistor" deviceset="R-EU_" device="R0603"/>
-<part name="R3" library="resistor" deviceset="R-EU_" device="R0603"/>
-<part name="R4" library="resistor" deviceset="R-EU_" device="R0603"/>
-<part name="R5" library="resistor" deviceset="R-EU_" device="R0603"/>
-<part name="R6" library="resistor" deviceset="R-EU_" device="R0603"/>
-<part name="R7" library="resistor" deviceset="R-EU_" device="R0603"/>
-<part name="R8" library="resistor" deviceset="R-EU_" device="R0603"/>
+<part name="R1" library="resistor" deviceset="R-EU_" device="R0603" value="10K"/>
+<part name="R2" library="resistor" deviceset="R-EU_" device="R0603" value="10K"/>
+<part name="R3" library="resistor" deviceset="R-EU_" device="R0603" value="10K"/>
+<part name="R4" library="resistor" deviceset="R-EU_" device="R0603" value="10K"/>
+<part name="R5" library="resistor" deviceset="R-EU_" device="R0603" value="10K"/>
+<part name="R6" library="resistor" deviceset="R-EU_" device="R0603" value="10K"/>
+<part name="R7" library="resistor" deviceset="R-EU_" device="R0603" value="10K"/>
+<part name="R8" library="resistor" deviceset="R-EU_" device="R0603" value="10K"/>
 <part name="P+27" library="SparkFun" deviceset="VCC" device=""/>
 <part name="P+28" library="SparkFun" deviceset="VCC" device=""/>
