File: controller-ha-v4.sch (EAGLE design)
At the start: 137 parts, among them U1 DS1307, U3 ARDUINO-MEGAFULL

Commit message: Submit all new design
Adding version 3-4 for driver & controller; Adding version 1-2 IO Module
Parts:
- removed ACDC: HLK-PM01, bontor:HLK-PM01
- removed AC_IN: AK3003, con-ptr500:AK3003
- removed C9-100N1, C9-100N10, C9-100N11, C9-100N12, C9-100N13, C9-100N14, C9-100N15, C9-100N16, C9-100N17, C9-100N18, C9-100N19, C9-100N2, C9-100N20, C9-100N21, C9-100N22, C9-100N23, C9-100N24, C9-100N25, C9-100N26, C9-100N3, C9-100N4, C9-100N5, C9-100N6, C9-100N7, C9-100N8, C9-100N9: (no value), rcl:C-EUC0603
- removed CN1: (no value), adafruit:DCBARRELPTH
- removed IN1, IN10, IN11, IN12, IN13, IN2, IN3, IN4, IN5, IN6, IN7, IN8, IN9, OUTA, OUTB, OUTC, OUTD, OUTE, OUTF, OUTG, OUTH, OUTI, OUTJ, OUTK, OUTL, OUTM: (no value), pinhead:PINHD-2X5
- removed JP1: (no value), pinhead:PINHD-1X4
- removed LED1, LED2: (no value), SparkFun-LED:LED-3MM-NO_SILK
- removed RN1, RN10, RN11, RN12, RN13, RN2, RN3, RN4, RN5, RN6, RN7, RN8, RN9: (no value), resistor-net:RN08
- removed SHIFT1, SHIFT10, SHIFT11, SHIFT12, SHIFT13, SHIFT2, SHIFT3, SHIFT4, SHIFT5, SHIFT6, SHIFT7, SHIFT8, SHIFT9: 74HC165D, 74xx-eu:74HC165D
- removed SHIFTOUTA, SHIFTOUTB, SHIFTOUTC, SHIFTOUTD, SHIFTOUTE, SHIFTOUTF, SHIFTOUTG, SHIFTOUTH, SHIFTOUTI, SHIFTOUTJ, SHIFTOUTK, SHIFTOUTL, SHIFTOUTM: 74HC595D, 74xx-eu:74HC595D
- added A-GRN, B-YLW: (no value), led:LEDCHIP-LED0805
- added IC2: LM358MX, linear:LM358MX
- added IN, OUT: (no value), adafruit:LEDCHIPLED_0805
- added JP4: (no value), SparkFun-Connectors:M05X2RA
- added MODE_SELECT: (no value), special:SW_DIP-2
- added NETLIGHT, STATUS: (no value), adafruit:LEDCHIP-LED0805
- added R1, R3, R4, R5: (no value), resistor:R-EU_R0805
- added U$3: 2.1MMJACKTHM, adafruit:2.1MMJACKTHM
- added U$6: 4-PIN-CON-1759017, maul:4-PIN-CON-1759017
- U$5: value SIMHOLDER3 -> SIM_HOLDER_PUSH; device SparkFun:SIMHOLDER3 -> maul:SIM_HOLDER_PUSH
- renumbered BAT to BAT1
Connections:
- removed net +9V: CN1.PWR, U$1.VIN
- removed net 1-1: IN1.1, RN1.5, SHIFT1A.A
- removed net 1-2: IN1.2, RN1.4, SHIFT1A.B
- removed net 1-3: IN1.3, RN1.3, SHIFT1A.C
- removed net 1-4: IN1.4, RN1.2, SHIFT1A.D
- removed net 1-5: IN1.5, RN1.6, SHIFT1A.E
- removed net 1-6: IN1.6, RN1.7, SHIFT1A.F
- removed net 1-7: IN1.7, RN1.8, SHIFT1A.G
- removed net 1-8: IN1.8, RN1.9, SHIFT1A.H
- removed net 10-1: IN10.1, RN10.5, SHIFT10A.A
- removed net 10-2: IN10.2, RN10.4, SHIFT10A.B
- removed net 10-3: IN10.3, RN10.3, SHIFT10A.C
- removed net 10-4: IN10.4, RN10.2, SHIFT10A.D
- removed net 10-5: IN10.5, RN10.6, SHIFT10A.E
- removed net 10-6: IN10.6, RN10.7, SHIFT10A.F
- removed net 10-7: IN10.7, RN10.8, SHIFT10A.G
- removed net 10-8: IN10.8, RN10.9, SHIFT10A.H
- removed net 11-1: IN11.1, RN11.5, SHIFT11A.A
- removed net 11-2: IN11.2, RN11.4, SHIFT11A.B
- removed net 11-3: IN11.3, RN11.3, SHIFT11A.C
- removed net 11-4: IN11.4, RN11.2, SHIFT11A.D
- removed net 11-5: IN11.5, RN11.6, SHIFT11A.E
- removed net 11-6: IN11.6, RN11.7, SHIFT11A.F
- removed net 11-7: IN11.7, RN11.8, SHIFT11A.G
- removed net 11-8: IN11.8, RN11.9, SHIFT11A.H
- removed net 12-1: IN12.1, RN12.5, SHIFT12A.A
- removed net 12-2: IN12.2, RN12.4, SHIFT12A.B
- removed net 12-3: IN12.3, RN12.3, SHIFT12A.C
- removed net 12-4: IN12.4, RN12.2, SHIFT12A.D
- removed net 12-5: IN12.5, RN12.6, SHIFT12A.E
- removed net 12-6: IN12.6, RN12.7, SHIFT12A.F
- removed net 12-7: IN12.7, RN12.8, SHIFT12A.G
- removed net 12-8: IN12.8, RN12.9, SHIFT12A.H
- removed net 13-1: IN13.1, RN13.5, SHIFT13A.A
- removed net 13-2: IN13.2, RN13.4, SHIFT13A.B
- removed net 13-3: IN13.3, RN13.3, SHIFT13A.C
- removed net 13-4: IN13.4, RN13.2, SHIFT13A.D
- removed net 13-5: IN13.5, RN13.6, SHIFT13A.E
- removed net 13-6: IN13.6, RN13.7, SHIFT13A.F
- removed net 13-7: IN13.7, RN13.8, SHIFT13A.G
- removed net 13-8: IN13.8, RN13.9, SHIFT13A.H
- removed net 2-1: IN2.1, RN2.5, SHIFT2A.A
- removed net 2-2: IN2.2, RN2.4, SHIFT2A.B
- removed net 2-3: IN2.3, RN2.3, SHIFT2A.C
- removed net 2-4: IN2.4, RN2.2, SHIFT2A.D
- removed net 2-5: IN2.5, RN2.6, SHIFT2A.E
- removed net 2-6: IN2.6, RN2.7, SHIFT2A.F
- removed net 2-7: IN2.7, RN2.8, SHIFT2A.G
- removed net 2-8: IN2.8, RN2.9, SHIFT2A.H
- removed net 3-1: IN3.1, RN3.5, SHIFT3A.A
- removed net 3-2: IN3.2, RN3.4, SHIFT3A.B
- removed net 3-3: IN3.3, RN3.3, SHIFT3A.C
- removed net 3-4: IN3.4, RN3.2, SHIFT3A.D
- removed net 3-5: IN3.5, RN3.6, SHIFT3A.E
- removed net 3-6: IN3.6, RN3.7, SHIFT3A.F
- removed net 3-7: IN3.7, RN3.8, SHIFT3A.G
- removed net 3-8: IN3.8, RN3.9, SHIFT3A.H
- removed net 4-1: IN4.1, RN4.5, SHIFT4A.A
- removed net 4-2: IN4.2, RN4.4, SHIFT4A.B
- removed net 4-3: IN4.3, RN4.3, SHIFT4A.C
- removed net 4-4: IN4.4, RN4.2, SHIFT4A.D
- removed net 4-5: IN4.5, RN4.6, SHIFT4A.E
- removed net 4-6: IN4.6, RN4.7, SHIFT4A.F
- removed net 4-7: IN4.7, RN4.8, SHIFT4A.G
- removed net 4-8: IN4.8, RN4.9, SHIFT4A.H
- removed net 5-1: IN5.1, RN5.5, SHIFT5A.A
- removed net 5-2: IN5.2, RN5.4, SHIFT5A.B
- removed net 5-3: IN5.3, RN5.3, SHIFT5A.C
- removed net 5-4: IN5.4, RN5.2, SHIFT5A.D
- removed net 5-5: IN5.5, RN5.6, SHIFT5A.E
- removed net 5-6: IN5.6, RN5.7, SHIFT5A.F
- removed net 5-7: IN5.7, RN5.8, SHIFT5A.G
- removed net 5-8: IN5.8, RN5.9, SHIFT5A.H
- removed net 6-1: IN6.1, RN6.5, SHIFT6A.A
- removed net 6-2: IN6.2, RN6.4, SHIFT6A.B
- removed net 6-3: IN6.3, RN6.3, SHIFT6A.C
- removed net 6-4: IN6.4, RN6.2, SHIFT6A.D
- removed net 6-5: IN6.5, RN6.6, SHIFT6A.E
- removed net 6-6: IN6.6, RN6.7, SHIFT6A.F
- removed net 6-7: IN6.7, RN6.8, SHIFT6A.G
- removed net 6-8: IN6.8, RN6.9, SHIFT6A.H
- removed net 7-1: IN7.1, RN7.5, SHIFT7A.A
- removed net 7-2: IN7.2, RN7.4, SHIFT7A.B
- removed net 7-3: IN7.3, RN7.3, SHIFT7A.C
- removed net 7-4: IN7.4, RN7.2, SHIFT7A.D
- removed net 7-5: IN7.5, RN7.6, SHIFT7A.E
- removed net 7-6: IN7.6, RN7.7, SHIFT7A.F
- removed net 7-7: IN7.7, RN7.8, SHIFT7A.G
- removed net 7-8: IN7.8, RN7.9, SHIFT7A.H
- removed net 8-1: IN8.1, RN8.5, SHIFT8A.A
- removed net 8-2: IN8.2, RN8.4, SHIFT8A.B
- removed net 8-3: IN8.3, RN8.3, SHIFT8A.C
- removed net 8-4: IN8.4, RN8.2, SHIFT8A.D
- removed net 8-5: IN8.5, RN8.6, SHIFT8A.E
- removed net 8-6: IN8.6, RN8.7, SHIFT8A.F
- removed net 8-7: IN8.7, RN8.8, SHIFT8A.G
- removed net 8-8: IN8.8, RN8.9, SHIFT8A.H
- removed net 9-1: IN9.1, RN9.5, SHIFT9A.A
- removed net 9-2: IN9.2, RN9.4, SHIFT9A.B
- removed net 9-3: IN9.3, RN9.3, SHIFT9A.C
- removed net 9-4: IN9.4, RN9.2, SHIFT9A.D
- removed net 9-5: IN9.5, RN9.6, SHIFT9A.E
- removed net 9-6: IN9.6, RN9.7, SHIFT9A.F
- removed net 9-7: IN9.7, RN9.8, SHIFT9A.G
- removed net 9-8: IN9.8, RN9.9, SHIFT9A.H
- removed net A-1: OUTA.1, SHIFTOUTAA.QA
- removed net A-2: OUTA.2, SHIFTOUTAA.QB
- removed net A-3: OUTA.3, SHIFTOUTAA.QC
- removed net A-4: OUTA.4, SHIFTOUTAA.QD
- removed net A-5: OUTA.5, SHIFTOUTAA.QE
- removed net A-6: OUTA.6, SHIFTOUTAA.QF
- removed net A-7: OUTA.7, SHIFTOUTAA.QG
- removed net A-8: OUTA.8, SHIFTOUTAA.QH
- removed net B-1: OUTB.1, SHIFTOUTBA.QA
- removed net B-2: OUTB.2, SHIFTOUTBA.QB
- removed net B-3: OUTB.3, SHIFTOUTBA.QC
- removed net B-4: OUTB.4, SHIFTOUTBA.QD
- removed net B-5: OUTB.5, SHIFTOUTBA.QE
- removed net B-6: OUTB.6, SHIFTOUTBA.QF
- removed net B-7: OUTB.7, SHIFTOUTBA.QG
- removed net B-8: OUTB.8, SHIFTOUTBA.QH
- removed net C-1: OUTC.1, SHIFTOUTCA.QA
- removed net C-2: OUTC.2, SHIFTOUTCA.QB
- removed net C-3: OUTC.3, SHIFTOUTCA.QC
- removed net C-4: OUTC.4, SHIFTOUTCA.QD
- removed net C-5: OUTC.5, SHIFTOUTCA.QE
- removed net C-6: OUTC.6, SHIFTOUTCA.QF
- removed net C-7: OUTC.7, SHIFTOUTCA.QG
- removed net C-8: OUTC.8, SHIFTOUTCA.QH
- removed net D-1: OUTD.1, SHIFTOUTDA.QA
- removed net D-2: OUTD.2, SHIFTOUTDA.QB
- removed net D-3: OUTD.3, SHIFTOUTDA.QC
- removed net D-4: OUTD.4, SHIFTOUTDA.QD
- removed net D-5: OUTD.5, SHIFTOUTDA.QE
- removed net D-6: OUTD.6, SHIFTOUTDA.QF
- removed net D-7: OUTD.7, SHIFTOUTDA.QG
- removed net D-8: OUTD.8, SHIFTOUTDA.QH
- removed net DBG_RX: U3.15(RX3)
- removed net DBG_TX: U3.14(TX3)
- removed net DS_OE: SHIFTOUTAA.G, SHIFTOUTBA.G, SHIFTOUTCA.G, SHIFTOUTDA.G, SHIFTOUTEA.G, SHIFTOUTFA.G, SHIFTOUTGA.G, SHIFTOUTHA.G, SHIFTOUTIA.G, SHIFTOUTJA.G, SHIFTOUTKA.G, SHIFTOUTLA.G, SHIFTOUTMA.G, U3.24
- removed net E-1: OUTE.1, SHIFTOUTEA.QA
- removed net E-2: OUTE.2, SHIFTOUTEA.QB
- removed net E-3: OUTE.3, SHIFTOUTEA.QC
- removed net E-4: OUTE.4, SHIFTOUTEA.QD
- removed net E-5: OUTE.5, SHIFTOUTEA.QE
- removed net E-6: OUTE.6, SHIFTOUTEA.QF
- removed net E-7: OUTE.7, SHIFTOUTEA.QG
- removed net E-8: OUTE.8, SHIFTOUTEA.QH
- removed net F-1: OUTF.1, SHIFTOUTFA.QA
- removed net F-2: OUTF.2, SHIFTOUTFA.QB
- removed net F-3: OUTF.3, SHIFTOUTFA.QC
- removed net F-4: OUTF.4, SHIFTOUTFA.QD
- removed net F-5: OUTF.5, SHIFTOUTFA.QE
- removed net F-6: OUTF.6, SHIFTOUTFA.QF
- removed net F-7: OUTF.7, SHIFTOUTFA.QG
- removed net F-8: OUTF.8, SHIFTOUTFA.QH
- removed net G-1: OUTG.1, SHIFTOUTGA.QA
- removed net G-2: OUTG.2, SHIFTOUTGA.QB
- removed net G-3: OUTG.3, SHIFTOUTGA.QC
- removed net G-4: OUTG.4, SHIFTOUTGA.QD
- removed net G-5: OUTG.5, SHIFTOUTGA.QE
- removed net G-6: OUTG.6, SHIFTOUTGA.QF
- removed net G-7: OUTG.7, SHIFTOUTGA.QG
- removed net G-8: OUTG.8, SHIFTOUTGA.QH
- removed net H-1: OUTH.1, SHIFTOUTHA.QA
- removed net H-2: OUTH.2, SHIFTOUTHA.QB
- removed net H-3: OUTH.3, SHIFTOUTHA.QC
- removed net H-4: OUTH.4, SHIFTOUTHA.QD
- removed net H-5: OUTH.5, SHIFTOUTHA.QE
- removed net H-6: OUTH.6, SHIFTOUTHA.QF
- removed net H-7: OUTH.7, SHIFTOUTHA.QG
- removed net H-8: OUTH.8, SHIFTOUTHA.QH
- removed net I-1: OUTI.1, SHIFTOUTIA.QA
- removed net I-2: OUTI.2, SHIFTOUTIA.QB
- removed net I-3: OUTI.3, SHIFTOUTIA.QC
- removed net I-4: OUTI.4, SHIFTOUTIA.QD
- removed net I-5: OUTI.5, SHIFTOUTIA.QE
- removed net I-6: OUTI.6, SHIFTOUTIA.QF
- removed net I-7: OUTI.7, SHIFTOUTIA.QG
- removed net I-8: OUTI.8, SHIFTOUTIA.QH
- removed net J-1: OUTJ.1, SHIFTOUTJA.QA
- removed net J-2: OUTJ.2, SHIFTOUTJA.QB
- removed net J-3: OUTJ.3, SHIFTOUTJA.QC
- removed net J-4: OUTJ.4, SHIFTOUTJA.QD
- removed net J-5: OUTJ.5, SHIFTOUTJA.QE
- removed net J-6: OUTJ.6, SHIFTOUTJA.QF
- removed net J-7: OUTJ.7, SHIFTOUTJA.QG
- removed net J-8: OUTJ.8, SHIFTOUTJA.QH
- removed net K-1: OUTK.1, SHIFTOUTKA.QA
- removed net K-2: OUTK.2, SHIFTOUTKA.QB
- removed net K-3: OUTK.3, SHIFTOUTKA.QC
- removed net K-4: OUTK.4, SHIFTOUTKA.QD
- removed net K-5: OUTK.5, SHIFTOUTKA.QE
- removed net K-6: OUTK.6, SHIFTOUTKA.QF
- removed net K-7: OUTK.7, SHIFTOUTKA.QG
- removed net K-8: OUTK.8, SHIFTOUTKA.QH
- removed net L-1: OUTL.1, SHIFTOUTLA.QA
- removed net L-2: OUTL.2, SHIFTOUTLA.QB
- removed net L-3: OUTL.3, SHIFTOUTLA.QC
- removed net L-4: OUTL.4, SHIFTOUTLA.QD
- removed net L-5: OUTL.5, SHIFTOUTLA.QE
- removed net L-6: OUTL.6, SHIFTOUTLA.QF
- removed net L-7: OUTL.7, SHIFTOUTLA.QG
- removed net L-8: OUTL.8, SHIFTOUTLA.QH
- removed net M-1: OUTM.1, SHIFTOUTMA.QA
- removed net M-2: OUTM.2, SHIFTOUTMA.QB
- removed net M-3: OUTM.3, SHIFTOUTMA.QC
- removed net M-4: OUTM.4, SHIFTOUTMA.QD
- removed net M-5: OUTM.5, SHIFTOUTMA.QE
- removed net M-6: OUTM.6, SHIFTOUTMA.QF
- removed net M-7: OUTM.7, SHIFTOUTMA.QG
- removed net M-8: OUTM.8, SHIFTOUTMA.QH
- removed net N$121: SHIFT10A.QH, SHIFT9A.SER
- removed net N$17: ACDC.AC_IN$2, AC_ING$1.KL
- removed net N$18: SHIFT2A.SER, SHIFT3A.QH
- removed net N$22: SHIFT4A.SER, SHIFT5A.QH
- removed net N$29: SHIFT11A.SER, SHIFT12A.QH
- removed net N$30: SHIFT10A.SER, SHIFT11A.QH
- removed net N$31: SHIFTOUTCA.QH*, SHIFTOUTDA.SER
- removed net N$32: SHIFTOUTEA.QH*, SHIFTOUTFA.SER
- removed net N$33: SHIFTOUTGA.QH*, SHIFTOUTHA.SER
- removed net N$34: SHIFTOUTIA.QH*, SHIFTOUTJA.SER
- removed net N$35: SHIFTOUTKA.QH*, SHIFTOUTLA.SER
- removed net N$36: SHIFT6A.SER, SHIFT7A.QH
- removed net N$37: SHIFTOUTBA.QH*, SHIFTOUTCA.SER
- removed net N$38: SHIFTOUTDA.QH*, SHIFTOUTEA.SER
- removed net N$39: SHIFTOUTFA.QH*, SHIFTOUTGA.SER
- removed net N$40: SHIFTOUTHA.QH*, SHIFTOUTIA.SER
- removed net N$41: SHIFTOUTJA.QH*, SHIFTOUTKA.SER
- removed net N$42: SHIFTOUTLA.QH*, SHIFTOUTMA.SER
- removed net N$50: SHIFT1A.SER, SHIFT2A.QH
- removed net N$7: ACDC.AC_IN$1, AC_ING$3.KL
- removed net RESET: R2.1
- new net +12V: U$1.VIN, U$2.VIN, U$3.TIP, U$6.4
- new net CTRL_SIMRESET: R2.1, U3.A2
- new net STATE_A: A-GRN.C, MODE_SELECT.3, U3.A3
- new net STATE_B: B-YLW.C, MODE_SELECT.4, U3.A4
- net CE: now also JP4.5, U3.6; no longer SHIFT10A.INH, SHIFT11A.INH, SHIFT12A.INH, SHIFT13A.INH, SHIFT1A.INH, SHIFT2A.INH, SHIFT3A.INH, SHIFT4A.INH, SHIFT5A.INH, SHIFT6A.INH, SHIFT7A.INH, SHIFT8A.INH, SHIFT9A.INH, U3.7
- net CLK: now also JP4.3, U3.7; no longer SHIFT10A.CLK, SHIFT11A.CLK, SHIFT12A.CLK, SHIFT13A.CLK, SHIFT1A.CLK, SHIFT2A.CLK, SHIFT3A.CLK, SHIFT4A.CLK, SHIFT5A.CLK, SHIFT6A.CLK, SHIFT7A.CLK, SHIFT8A.CLK, SHIFT9A.CLK, U3.6
- net GND: now also IC1.GND@3, IC2P.V-, IN.C, JP4.2, JP4.9, MODE_SELECT.1, MODE_SELECT.2, OUT.C, U$3.RING, U$3.RING_SW, U$5.5, U$6.2, U$6.3; no longer ACDC.GND, C9-100N1.1, C9-100N10.1, C9-100N11.1, C9-100N12.1, C9-100N13.1, C9-100N14.1, C9-100N15.1, C9-100N16.1, C9-100N17.1, C9-100N18.1, C9-100N19.1, C9-100N2.1, C9-100N20.1, C9-100N21.1, C9-100N22.1, C9-100N23.1, C9-100N24.1, C9-100N25.1, C9-100N26.1, C9-100N3.1, C9-100N4.1, C9-100N5.1, C9-100N6.1, C9-100N7.1, C9-100N8.1, C9-100N9.1, CN1.GND, CN1.GNDBREAK, IN1.10, IN10.10, IN11.10, IN12.10, IN13.10, IN2.10, IN3.10, IN4.10, IN5.10, IN6.10, IN7.10, IN8.10, IN9.10, JP1.3, JP1.4, OUTA.10, OUTB.10, OUTC.10, OUTD.10, OUTE.10, OUTF.10, OUTG.10, OUTH.10, OUTI.10, OUTJ.10, OUTK.10, OUTL.10, OUTM.10, SHIFT10P.GND, SHIFT11P.GND, SHIFT12P.GND, SHIFT13P.GND, SHIFT1P.GND, SHIFT2P.GND, SHIFT3P.GND, SHIFT4P.GND, SHIFT5P.GND, SHIFT6P.GND, SHIFT7P.GND, SHIFT8P.GND, SHIFT9P.GND, U$5.GND
- net N$11: now also NETLIGHT.A; no longer LED2.A
- net N$12: now also NETLIGHT.C; no longer LED2.C
- net N$21: now also IC2A.+IN, IC2A.OUT, R1.1; no longer SHIFT3A.SER, SHIFT4A.QH
- net N$24: now also IC2B.+IN, IC2B.OUT, R3.1; no longer SHIFT5A.SER, SHIFT6A.QH
- net N$25: now also OUT.A, R1.2; no longer SHIFT7A.SER, SHIFT8A.QH
- net N$26: now also IN.A, R3.2; no longer SHIFTOUTAA.QH*, SHIFTOUTBA.SER
- net N$27: now also A-GRN.A, R4.1; no longer SHIFT8A.SER, SHIFT9A.QH
- net N$28: now also B-YLW.A, R5.1; no longer SHIFT12A.SER, SHIFT13A.QH
- net N$8: now also STATUS.A; no longer LED1.A
- net N$9: now also STATUS.C; no longer LED1.C
- net PL: now also JP4.7, U3.5; no longer SHIFT10A.SH/!LD, SHIFT11A.SH/!LD, SHIFT12A.SH/!LD, SHIFT13A.SH/!LD, SHIFT1A.SH/!LD, SHIFT2A.SH/!LD, SHIFT3A.SH/!LD, SHIFT4A.SH/!LD, SHIFT5A.SH/!LD, SHIFT6A.SH/!LD, SHIFT7A.SH/!LD, SHIFT8A.SH/!LD, SHIFT9A.SH/!LD, U3.8
- net Q7: now also IC2A.-IN, JP4.1, U3.8; no longer SHIFT1A.QH, U3.5
- net SHCP: now also JP4.8; no longer SHIFTOUTAA.SCK, SHIFTOUTBA.SCK, SHIFTOUTCA.SCK, SHIFTOUTDA.SCK, SHIFTOUTEA.SCK, SHIFTOUTFA.SCK, SHIFTOUTGA.SCK, SHIFTOUTHA.SCK, SHIFTOUTIA.SCK, SHIFTOUTJA.SCK, SHIFTOUTKA.SCK, SHIFTOUTLA.SCK, SHIFTOUTMA.SCK
- net SR_DS: now also IC2B.-IN, JP4.4; no longer SHIFTOUTAA.SER
- net SR_RST: now also JP4.10, U3.15(RX3); no longer SHIFTOUTAA.SCL, SHIFTOUTBA.SCL, SHIFTOUTCA.SCL, SHIFTOUTDA.SCL, SHIFTOUTEA.SCL, SHIFTOUTFA.SCL, SHIFTOUTGA.SCL, SHIFTOUTHA.SCL, SHIFTOUTIA.SCL, SHIFTOUTJA.SCL, SHIFTOUTKA.SCL, SHIFTOUTLA.SCL, SHIFTOUTMA.SCL, U3.19(RX1)
- net STCP: now also JP4.6; no longer SHIFTOUTAA.RCK, SHIFTOUTBA.RCK, SHIFTOUTCA.RCK, SHIFTOUTDA.RCK, SHIFTOUTEA.RCK, SHIFTOUTFA.RCK, SHIFTOUTGA.RCK, SHIFTOUTHA.RCK, SHIFTOUTIA.RCK, SHIFTOUTJA.RCK, SHIFTOUTKA.RCK, SHIFTOUTLA.RCK, SHIFTOUTMA.RCK
- net USIM_CLK: now also U$5.3; no longer U$5.CLK
- net USIM_DATA: now also U$5.7; no longer U$5.I/O
- net USIM_RESET: now also U$5.2; no longer U$5.RST
- net USIM_VCC: now also U$5.1; no longer U$5.VCC
- net VCC: now also IC2P.V+, R4.2, R5.2, U$6.1; no longer ACDC.VOUT, C9-100N1.2, C9-100N10.2, C9-100N11.2, C9-100N12.2, C9-100N13.2, C9-100N14.2, C9-100N15.2, C9-100N16.2, C9-100N17.2, C9-100N18.2, C9-100N19.2, C9-100N2.2, C9-100N20.2, C9-100N21.2, C9-100N22.2, C9-100N23.2, C9-100N24.2, C9-100N25.2, C9-100N26.2, C9-100N3.2, C9-100N4.2, C9-100N5.2, C9-100N6.2, C9-100N7.2, C9-100N8.2, C9-100N9.2, IN1.9, IN10.9, IN11.9, IN12.9, IN13.9, IN2.9, IN3.9, IN4.9, IN5.9, IN6.9, IN7.9, IN8.9, IN9.9, JP1.1, JP1.2, OUTA.9, OUTB.9, OUTC.9, OUTD.9, OUTE.9, OUTF.9, OUTG.9, OUTH.9, OUTI.9, OUTJ.9, OUTK.9, OUTL.9, OUTM.9, RN1.1, RN10.1, RN11.1, RN12.1, RN13.1, RN2.1, RN3.1, RN4.1, RN5.1, RN6.1, RN7.1, RN8.1, RN9.1, SHIFT10P.VCC, SHIFT11P.VCC, SHIFT12P.VCC, SHIFT13P.VCC, SHIFT1P.VCC, SHIFT2P.VCC, SHIFT3P.VCC, SHIFT4P.VCC, SHIFT5P.VCC, SHIFT6P.VCC, SHIFT7P.VCC, SHIFT8P.VCC, SHIFT9P.VCC, U$2.VIN
Other:
- note removed: "Input Signals"
- note removed: "Output Signals"
- note removed: "SUPPLY AC/DC"
- note removed: "WiFi"
- note removed: "Wifi Comunication"
- moved on the sheet: D15, R26-1K, R27-1K, R28-10K, T2

Commit message: change in controller design
Change component position & adding hole to controller design
Parts:
- added JP1, JP2, JP3, JP5, JP6: (no value), adafruit:PINHD-1X8CLEANBIG
- added JP7: (no value), pinhead:PINHD-2X18
- added JP8: (no value), adafruit:PINHD-1X6CB
- A-GRN, IN, NETLIGHT, OUT: value (none) -> green
- B-YLW, STATUS: value (none) -> yellow
- C10-4U7: value (none) -> 4.7nF
- C11, CSIM_22P: value (none) -> 22pF
- C7-100U, C8-100U: value (none) -> 100uF
- C9, CSIM_100N: value (none) -> 100nF
- R1, R3: value (none) -> 220
- R1-1K, R1-1K1, R20-1K, R23-1K, R26-1K, R27-1K, R4, R5: value (none) -> 1K
- R10-22, R11-22, R9-22: value (none) -> 22
- R2, R30: value R120 -> 120
- R25-10K, R28-10K: value (none) -> 10K
- R2K2_SCL, R2K2_SDA: value (none) -> 2.2K
- R5-2K, R5-2K1: value (none) -> 2K
- renumbered C11-22P to C11, C9-100N to C9, U$1 to DC2DC-2, U$2 to DC2DC-1, U$3 to DC_JACKTHM, U$4 to ESP8266, U$5 to SIM_HOLDER, U$6 to 4-WAY_L-TERMINAL, U3 to ARDUINO_FOOTPRINT
