File: IO_board-ha-v3.sch (EAGLE design)
At the start: 43 parts, among them J1 4-PIN-CON-1759017, J2 4-PIN-CON-1759017

Commit message: Revising Controller & IO Module
Some module (SIM900 & RTC) are not working, IO Module suddenly shorted
Parts:
- removed C1, C10, C2, C4, C5, C6, C7, C9: 100nF, resistor:C-EUC0805
Connections:
- removed net SR_RST: JP1.10, JP2.10, SHIFTOUTAA.SCL, SHIFTOUTBA.SCL, SHIFTOUTCA.SCL, SHIFTOUTDA.SCL, SHIFTOUTEA.SCL
- net +12V: no longer C10.2, C6.2, C7.2, C9.2
- net GND: no longer C1.2, C10.1, C2.2, C4.2, C5.2, C6.1, C7.1, C9.1
- net VCC: now also JP1.10, JP2.10, SHIFTOUTAA.SCL, SHIFTOUTBA.SCL, SHIFTOUTCA.SCL, SHIFTOUTDA.SCL, SHIFTOUTEA.SCL; no longer C1.1, C2.1, C4.1, C5.1
