File: IO_board-ha-v3-rev1.sch (EAGLE design)
At the start: 47 parts, among them J1 4-PIN-CON-1759017, J2 4-PIN-CON-1759017

Commit message: Upgrade to version 5
With LAN Ethernet ENC28J60; adding relay for restarting 12V modules
(Driver & IO).
Parts:
- added 12V, 5V: (no value), SparkFun-LED:LED3MM
- added R10: 220, rcl:R-EU_R0805
- added R9: 1k, rcl:R-EU_R0805
Connections:
- new net N$13: 12V.C, R9.1
- new net N$17: 5V.C, R10.1
- net +12V: now also 12V.A
- net GND: now also R10.2, R9.2
- net VCC: now also 5V.A
Other:
- note added: "Command_DC_Signal"
- note added: "Out_to_Driver"
- note added: "Power_Indicators"
- note added: "Power_Socket_4Pins"
- note added: "Switching_Power_Supply"
- moved on the sheet: JP1, JP2, R1, R2, R3, R4, R5, R6, R7, R8, RN1, RN2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
