File: controller-ha-v5.sch (EAGLE design)
At the start: 29 parts, among them IC2 LM358MX, U1 DS1307

Commit message: autoroute
remove gnd plane, add gnd route
Connections:
- net AUTORESET: now also ARDUINO_FOOTPRINT.A5
Changed lines of the file:
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@@
 <wire x1="220.98" y1="91.44" x2="233.68" y2="91.44" width="0.1524" layer="91"/>
+</segment>
+<segment>
+<pinref part="ARDUINO_FOOTPRINT" gate="G$1" pin="A5"/>
+<wire x1="294.64" y1="93.98" x2="292.1" y2="93.98" width="0.1524" layer="91"/>
+<label x="292.1" y="93.98" size="1.27" layer="95" rot="R180" xref="yes"/>
 </segment>
 </net>

Commit message: Upgrade to version 5
With LAN Ethernet ENC28J60; adding relay for restarting 12V modules
(Driver & IO).
Parts:
- removed C4: 100uF 35V, resistor:CPOL-US153CLV-0605
- removed R14: 120k, rcl:R-EU_R0805
- removed RST_S: (no value), adafruit:PINHD-1X3CB
- added C5: 100uF 16V, resistor:CPOL-US153CLV-0605
- added D1: (no value), adafruit:DIODESMA
- added K1: M3XXH, relay:M3XXH
- added R16: 120k, rcl:R-EU_R0805
- added R17: 10k, rcl:R-EU_R0805
- added R18: 1k, rcl:R-EU_R0805
- added R2: 10K, resistor:R-EU_R0805
- added RST_S1: (no value), adafruit:PINHD-1X3CB
- added T2, T3: (no value), transistor:MMBT2222ALT1-NPN-SOT23-BEC
Connections:
- new net DRV_ON: ARDUINO_FOOTPRINT.14(TX3), T2.B
- new net N$3: 4-WAY_L-TERMINAL.1, 4-WAY_L-TERMINAL.4, K12.P
- new net N$4: D1.A, K11.2, R2.1, T2.C
- new net N$5: R17.2, RST_S1.3, T3.E
- new net NET1: C5.+, R16.1, R18.2, T3.B
- net +12V: now also D1.C, K11.1, K12.O, R2.2; no longer 4-WAY_L-TERMINAL.1, 4-WAY_L-TERMINAL.4
- net AUTORESET: now also R18.1; no longer C4.+, R14.1, RST_S.3
- net GND: now also C5.-, R17.1, T2.E; no longer C4.-
- net NC: now also RST_S1.1; no longer RST_S.1
- net RST: now also RST_S1.2; no longer RST_S.2
- net VCC: now also R16.2, T3.C; no longer R14.2
